Commit message: Jan 11th

File: ros_dd/urdf/ros_dd.urdf (robot description, URDF)
Before this commit: robot ros_dd, 2 links, 1 joints
Links:
- added link wheel2_link; visual cylinder length=0.1 radius=0.15
- added link wheel3_link; visual cylinder length=0.1 radius=0.15
- added link wheel4_link; visual cylinder length=0.1 radius=0.15
Joints:
- added joint wheel2_joint: type continuous, parent body_link, child wheel2_link, origin xyz=-0.3 0.35 -0.1 rpy=0 0 0, axis 0 1 0
- added joint wheel3_joint: type continuous, parent body_link, child wheel3_link, origin xyz=0.3 -0.35 -0.1 rpy=0 0 0, axis 0 1 0
- added joint wheel4_joint: type continuous, parent body_link, child wheel4_link, origin xyz=0.3 0.35 -0.1 rpy=0 0 0, axis 0 1 0
