Commit message: Nov 13

File: ros_dd_simulation/ros_dd_gazebo/urdf/ros_dd.urdf (robot description, URDF)
Before this commit: robot ros_dd_small, 6 links, 5 joints
Links:
- removed link body_link
- removed link wheel1_link
- removed link wheel2_link
- removed link wheel3_link
- removed link wheel4_link
- added link base_footprint
- added link base_link, mass 3.0; collision box size=0.5 0.3 0.15; visual box size=0.5 0.3 0.15
- added link caster_link_front, mass 0.03; collision sphere radius=0.03; visual sphere radius=0.03
- added link caster_link_rear, mass 0.03; collision sphere radius=0.03; visual sphere radius=0.03
- added link left_wheel_link, mass 0.0625; collision cylinder length=0.05 radius=0.075; visual cylinder length=0.05 radius=0.075
- added link right_wheel_link, mass 0.0625; collision cylinder length=0.05 radius=0.075; visual cylinder length=0.05 radius=0.075
- link laser_link: mass 0.0125 -> 0.05
Joints:
- removed joint wheel1_joint
- removed joint wheel2_joint
- removed joint wheel3_joint
- removed joint wheel4_joint
- added joint base_joint: type fixed, parent base_footprint, child base_link, origin xyz=0 0 0.075 rpy=0 0 0
- added joint caster_front_joint: type fixed, parent base_link, child caster_link_front, origin xyz=0.2 -0.0 -0.005 rpy=0 0 0
- added joint caster_rear_joint: type fixed, parent base_link, child caster_link_rear, origin xyz=-0.2 -0.0 -0.005 rpy=0 0 0
- added joint left_wheel_joint: type continuous, parent base_link, child left_wheel_link, origin xyz=0 0.175 -0.008 rpy=0 0 0, axis 0 1 0
- added joint right_wheel_joint: type continuous, parent base_link, child right_wheel_link, origin xyz=0 -0.175 -0.008 rpy=0 0 0, axis 0 1 0
- joint laser_joint: origin xyz=0.225 0 0.125 rpy=0 0 0 -> xyz=0.3 0 0.15 rpy=0 0 0; parent body_link -> base_link
